File: eagle/gas-sensor.sch (EAGLE design)
At the start: 41 parts, among them CON1 SPI, IC1 MCP1703CB, J2 RJ12RIGHTANGLE-I2C, J3 RJ12RIGHTANGLE-I2C, U1 ATMEGA328P_TQFP, U2 HX711, X1 8MHz

Commit message: description of new project
Parts:
- removed C6: 100nF, rcl:C-EUC0805K
- removed S1: Reset, Testing:SWITCH-MOMENTARY-2SMD-ALT01
- removed SJ2: A1, jumper:SJ
Connections:
- net A7: no longer SJ2.1
- net DTR: no longer C6.1
- net GND: no longer S1.1, SJ2.2
- net RESET: no longer C6.2, S1.2
