File: kicad/gas-sensor.sch (KiCad schematic (older format))
At the start: 26 parts, among them J1 RJ12, U1 DS18B20, U2 FT232RL, U3 MCP1703A-3302_SOT23, U4 ATmega328P-AU, U5 DHT22, Y1 8MHz

Commit message: First version of PCB
with 3D components
Parts:
- removed C1: 100nF, Capacitor_SMD:C_0805_2012Metric_Pad1.15x1.40mm_HandSolder, symbol Device:C
- removed C5: 10u, Capacitor_SMD:C_0805_2012Metric_Pad1.15x1.40mm_HandSolder, symbol Device:C
- removed U2: FT232RL, Package_SO:SSOP-28_5.3x10.2mm_P0.65mm, symbol Interface_USB:FT232RL
- removed U3: MCP1703A-3302_SOT23, Package_TO_SOT_SMD:SOT-23, symbol Regulator_Linear:MCP1703A-3302_SOT23
- added J2: Conn FT232RL, Connector_PinHeader_2.54mm:PinHeader_1x06_P2.54mm_Vertical, symbol Connector:Conn_01x06_Female
- added J3: PJ-017DH, gas_sensor:PC-017C, symbol gas_sensor:PJ-017DH
- added Q1, Q2: BSP75, Package_TO_SOT_SMD:SOT-223-3_TabPin2, symbol gas_sensor:BSP75
Connections:
- net labels added: Sensor1_ON, Sensor2, Sensor2_ON
- net labels removed: +3.3V, +BATT, Sensor4
- wire segments 152 -> 140
- no-connect marks 7 -> 8
Other:
- moved on the sheet: C6, C7, GS1, GS3, GS4, R3, R4, SP1

Commit message: update
Parts:
- removed J3: PJ-017DH, gas_sensor:PC-017C, symbol gas_sensor:PJ-017DH
- added C1: 100nF, Capacitor_SMD:C_0805_2012Metric_Pad1.15x1.40mm_HandSolder, symbol Device:C
- added J3: 5V_Power_source, Connector_BarrelJack:BarrelJack_Horizontal, symbol Connector:Conn_Coaxial_Power
- added J4, J5, J6, J7: hole, MountingHole:MountingHole_3.2mm_M3, symbol Connector:Conn_01x01_Female
- added R5: R, Capacitor_SMD:C_0805_2012Metric_Pad1.15x1.40mm_HandSolder, symbol Device:R
- GS1: symbol gas_sensor:MQ-4 -> gas-sensor-rescue:MQ-4-gas_sensor
- GS3: symbol gas_sensor:MQ-8 -> gas-sensor-rescue:MQ-8-gas_sensor
- GS4: symbol gas_sensor:MH-Z19 -> gas-sensor-rescue:MH-Z19-gas_sensor
- Q1, Q2: symbol gas_sensor:BSP75 -> gas-sensor-rescue:BSP75-gas_sensor
- SP1: symbol gas_sensor:ICSP -> gas-sensor-rescue:ICSP-gas_sensor
- U5: symbol gas_sensor:DHT22 -> gas-sensor-rescue:DHT22-gas_sensor
- Y1: footprint Crystal:Crystal_SMD_0603-2Pin_6.0x3.5mm_HandSoldering -> Crystal:Crystal_SMD_5032-2Pin_5.0x3.2mm_HandSoldering
Connections:
- net MISO is gone; now on net LCD_RW: SP1.1 (MISO), U4.16 (PB4)
- net MOSI is gone; now on net LCD_E: SP1.4 (MOSI), U4.15 (PB3)
- net SCK is gone; now on net LCD_RS: SP1.3 (SCK), U4.17 (PB5)
- net +5V: now also U1.3 (VDD), J3.1 (In)
- net GND: now also C1.2, J3.2 (Ext)
- net VCC: now also DS1.3 (VO), C1.1; no longer DS1.15 (LED(+)), U1.3 (VDD)
- net LCD_RS: now reaches DS1.4 (RS)
- net LCD_RW: now reaches DS1.5 (R/W)
- net LCD_E: now reaches DS1.6 (E)
- new net: DS1.15 (LED(+)), R5.2
- new net LCD_LED: R5.1
- no-connect marks 8 -> 12
Other:
- note removed: "PAS FINI BRANCHEMENT LCD\n"

Commit message: Update
Parts:
- removed R5: R, Capacitor_SMD:C_0805_2012Metric_Pad1.15x1.40mm_HandSolder, symbol Device:R
- added R2: R, Resistor_SMD:R_0805_2012Metric_Pad1.15x1.40mm_HandSolder, symbol Device:R
- GS1: symbol gas-sensor-rescue:MQ-4-gas_sensor -> gas_sensor:MQ-4
- GS2: renamed from GS3; symbol gas-sensor-rescue:MQ-8-gas_sensor -> gas_sensor:MQ-8
- GS3: renamed from GS4; symbol gas-sensor-rescue:MH-Z19-gas_sensor -> gas_sensor:MH-Z19
- Q1, Q2: symbol gas-sensor-rescue:BSP75-gas_sensor -> BSP75:BSP75
- SP1: symbol gas-sensor-rescue:ICSP-gas_sensor -> ICSP:ICSP
- U3: renamed from U5; symbol gas-sensor-rescue:DHT22-gas_sensor -> gas_sensor:DHT22
- renumbered C3 to C1, C4 to C2, C6 to C3, C7 to C4, C1 to C5, C2 to C6, J2 to J1, J1 to J2, J4 to J3, J5 to J4, J6 to J5, J7 to J6, J3 to J7, R2 to R1, R1 to R3, R3 to R4, R4 to R5, U4 to U2
Connections:
- net HUM: now also U2.2 (PD4); no longer U2.26 (PC3)
- net LCD1: now also U2.14 (PB2); no longer U2.11 (PD7)
- net LCD_E: now also U2.12 (PB0); no longer SP1.4 (MOSI), U2.15 (PB3)
- net LCD_LED: now also U2.13 (PB1), R2.1
- net LCD_RS: now also U2.10 (PD6); no longer SP1.3 (SCK), U2.17 (PB5)
- net LCD_RW: now also U2.11 (PD7); no longer SP1.1 (MISO), U2.16 (PB4)
- net PWM_MH-Z19: now also U2.1 (PD3); no longer U2.9 (PD5)
- net RX_MH-Z19: now also U2.26 (PC3); no longer U2.32 (PD2)
- net Sensor1: now also U2.19 (ADC6); no longer U2.25 (PC2)
- net Sensor1_ON: now also U2.22 (ADC7); no longer U2.13 (PB1)
- net Sensor2: now also U2.23 (PC0); no longer U2.19 (ADC6)
- net Sensor2_ON: now also U2.24 (PC1); no longer U2.1 (PD3)
- net Sensor3: now also U2.32 (PD2); no longer U2.22 (ADC7)
- net TEMP: now also U2.9 (PD5); no longer U2.10 (PD6)
- net TX_MH-Z19: now also U2.25 (PC2); no longer U2.2 (PD4)
- net at DS1.15 (LED(+)): now also R2.2
- net LCD2 renamed LCD2_MOSI
- net LCD2_MOSI: now also SP1.4 (MOSI), U2.15 (PB3); no longer U2.12 (PB0)
- net LCD3 renamed LCD3_MISO
- net LCD3_MISO: now also SP1.1 (MISO), U2.16 (PB4); no longer U2.23 (PC0)
- net LCD4 renamed LCD4_SCK
- net LCD4_SCK: now also SP1.3 (SCK), U2.17 (PB5); no longer U2.24 (PC1)
- no-connect marks 12 -> 11

Commit message: Update
Parts:
- added J10, J11, J8, J9: hole, MountingHole:MountingHole_3.2mm_M3, symbol Connector:Conn_01x01_Female
Connections:
- no-connect marks 11 -> 15
Other:
- moved on the sheet: J3, J4, J5, J6
Changed lines of the file:
@@
 L Connector:Conn_01x01_Female J3
 U 1 1 5C8A50EC
-P 3200 2400
-F 0 "J3" H 3227 2426 50  0000 L CNN
-F 1 "hole" H 3227 2335 50  0000 L CNN
-F 2 "MountingHole:MountingHole_3.2mm_M3" H 3200 2400 50  0001 C CNN
-F 3 "~" H 3200 2400 50  0001 C CNN
-	1    3200 2400
+P 3550 2450
+F 0 "J3" H 3577 2476 50  0000 L CNN
+F 1 "hole" H 3577 2385 50  0000 L CNN
+F 2 "MountingHole:MountingHole_3.2mm_M3" H 3550 2450 50  0001 C CNN
+F 3 "~" H 3550 2450 50  0001 C CNN
+	1    3550 2450
 	1    0    0    -1
 $EndComp
-NoConn ~ 3000 2400
+NoConn ~ 3350 2450
 $Comp
 L Connector:Conn_01x01_Female J4
 U 1 1 5C8C9BF5
-P 3200 2600
-F 0 "J4" H 3227 2626 50  0000 L CNN
-F 1 "hole" H 3227 2535 50  0000 L CNN
-F 2 "MountingHole:MountingHole_3.2mm_M3" H 3200 2600 50  0001 C CNN
-F 3 "~" H 3200 2600 50  0001 C CNN
-	1    3200 2600
+P 3550 2650
+F 0 "J4" H 3577 2676 50  0000 L CNN
+F 1 "hole" H 3577 2585 50  0000 L CNN
+F 2 "MountingHole:MountingHole_3.2mm_M3" H 3550 2650 50  0001 C CNN
+F 3 "~" H 3550 2650 50  0001 C CNN
+	1    3550 2650
 	1    0    0    -1
 $EndComp
@@
 L Connector:Conn_01x01_Female J5
 U 1 1 5C8C9C43
-P 3200 2800
-F 0 "J5" H 3227 2826 50  0000 L CNN
-F 1 "hole" H 3227 2735 50  0000 L CNN
-F 2 "MountingHole:MountingHole_3.2mm_M3" H 3200 2800 50  0001 C CNN
-F 3 "~" H 3200 2800 50  0001 C CNN
-	1    3200 2800
+P 3550 2850
+F 0 "J5" H 3577 2876 50  0000 L CNN
+F 1 "hole" H 3577 2785 50  0000 L CNN
+F 2 "MountingHole:MountingHole_3.2mm_M3" H 3550 2850 50  0001 C CNN
+F 3 "~" H 3550 2850 50  0001 C CNN
+	1    3550 2850
 	1    0    0    -1
 $EndComp
@@
 L Connector:Conn_01x01_Female J6
 U 1 1 5C8C9C9B
-P 3200 3000
-F 0 "J6" H 3227 3026 50  0000 L CNN
-F 1 "hole" H 3227 2935 50  0000 L CNN
-F 2 "MountingHole:MountingHole_3.2mm_M3" H 3200 3000 50  0001 C CNN
-F 3 "~" H 3200 3000 50  0001 C CNN
-	1    3200 3000
+P 3550 3050
+F 0 "J6" H 3577 3076 50  0000 L CNN
+F 1 "hole" H 3577 2985 50  0000 L CNN
+F 2 "MountingHole:MountingHole_3.2mm_M3" H 3550 3050 50  0001 C CNN
+F 3 "~" H 3550 3050 50  0001 C CNN
+	1    3550 3050
 	1    0    0    -1
 $EndComp
-NoConn ~ 3000 2600
-NoConn ~ 3000 2800
-NoConn ~ 3000 3000
+NoConn ~ 3350 2650
+NoConn ~ 3350 2850
+NoConn ~ 3350 3050
 Wire Wire Line
 	4550 6100 4450 6100
@@
 Wire Wire Line
 	6500 3000 6800 3000
+$Comp
+L Connector:Conn_01x01_Female J8
+U 1 1 5C897406
+P 3100 2450
+F 0 "J8" H 3127 2476 50  0000 L CNN
+F 1 "hole" H 3127 2385 50  0000 L CNN
+F 2 "MountingHole:MountingHole_3.2mm_M3" H 3100 2450 50  0001 C CNN
+F 3 "~" H 3100 2450 50  0001 C CNN
+	1    3100 2450
+	1    0    0    -1
+$EndComp
+$Comp
+L Connector:Conn_01x01_Female J9
+U 1 1 5C897463
+P 3100 2650
+F 0 "J9" H 3127 2676 50  0000 L CNN
+F 1 "hole" H 3127 2585 50  0000 L CNN
+F 2 "MountingHole:MountingHole_3.2mm_M3" H 3100 2650 50  0001 C CNN
+F 3 "~" H 3100 2650 50  0001 C CNN
+	1    3100 2650
+	1    0    0    -1
+$EndComp
+$Comp
+L Connector:Conn_01x01_Female J10
+U 1 1 5C8974BE
+P 3100 2850
+F 0 "J10" H 3127 2876 50  0000 L CNN
+F 1 "hole" H 3127 2785 50  0000 L CNN
+F 2 "MountingHole:MountingHole_3.2mm_M3" H 3100 2850 50  0001 C CNN
+F 3 "~" H 3100 2850 50  0001 C CNN
+	1    3100 2850
+	1    0    0    -1
+$EndComp
+$Comp
+L Connector:Conn_01x01_Female J11
+U 1 1 5C89751A
+P 3100 3050
+F 0 "J11" H 3127 3076 50  0000 L CNN
+F 1 "hole" H 3127 2985 50  0000 L CNN
+F 2 "MountingHole:MountingHole_3.2mm_M3" H 3100 3050 50  0001 C CNN
+F 3 "~" H 3100 3050 50  0001 C CNN
+	1    3100 3050
+	1    0    0    -1
+$EndComp
+NoConn ~ 2900 2450
+NoConn ~ 2900 2650
+NoConn ~ 2900 2850
+NoConn ~ 2900 3050
 $EndSCHEMATC
