File: kicad/gas-sensor.sch (KiCad schematic (older format))
At the start: 41 parts, among them J1 Conn FT232RL, J10 hole, J11 hole, J2 RJ12, J3 hole, J4 hole, J5 hole, J6 hole, J7 5V_Power_source, J8 hole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

Commit message: Update CAD
Parts:
- removed J10, J11, J8, J9: hole, MountingHole:MountingHole_3.2mm_M3, symbol Connector:Conn_01x01_Female
- Q1, Q2: footprint Package_TO_SOT_SMD:SOT-223-3_TabPin2 -> Package_TO_SOT_SMD:SOT-223-3_TabPin3
Connections:
- net GND: now also Q1.3 (S), Q2.3 (S); no longer Q1.2 (D), Q2.2 (D)
- net at GS1.6 (H): now also Q1.2 (D); no longer Q1.3 (S)
- net at GS2.6 (H): now also Q2.2 (D); no longer Q2.3 (S)
- no-connect marks 16 -> 12
Other:
- moved on the sheet: Q1, Q2, R4, R5
Changed lines of the file:
@@
 L Device:R R5
 U 1 1 5C636C21
-P 9300 4100
-F 0 "R5" H 9370 4146 50  0000 L CNN
-F 1 "10k" H 9370 4055 50  0000 L CNN
-F 2 "Resistor_SMD:R_0805_2012Metric_Pad1.15x1.40mm_HandSolder" V 9230 4100 50  0001 C CNN
-F 3 "~" H 9300 4100 50  0001 C CNN
-	1    9300 4100
+P 9100 4100
+F 0 "R5" H 9170 4146 50  0000 L CNN
+F 1 "10k" H 9170 4055 50  0000 L CNN
+F 2 "Resistor_SMD:R_0805_2012Metric_Pad1.15x1.40mm_HandSolder" V 9030 4100 50  0001 C CNN
+F 3 "~" H 9100 4100 50  0001 C CNN
+	1    9100 4100
 	1    0    0    -1
 $EndComp
@@
 L BSP75:BSP75 Q1
 U 1 1 5C925971
-P 10000 2350
-F 0 "Q1" H 10206 2396 50  0000 L CNN
-F 1 "BSP75" H 10206 2305 50  0000 L CNN
-F 2 "Package_TO_SOT_SMD:SOT-223-3_TabPin2" H 10200 2275 50  0001 L CIN
-F 3 "" H 10200 2425 50  0001 L CNN
-	1    10000 2350
-	-1   0    0    1
+P 9800 2350
+F 0 "Q1" H 10006 2396 50  0000 L CNN
+F 1 "BSP75" H 10006 2305 50  0000 L CNN
+F 2 "Package_TO_SOT_SMD:SOT-223-3_TabPin3" H 10000 2275 50  0001 L CIN
+F 3 "" H 10000 2425 50  0001 L CNN
+	1    9800 2350
+	1    0    0    -1
 $EndComp
 Wire Wire Line
 	9900 2150 9900 2100
-Text HLabel 10450 2350 2    50   Input ~ 0
+Text HLabel 9450 2350 1    50   Input ~ 0
 Sensor1_ON
 $Comp
@@
 L BSP75:BSP75 Q2
 U 1 1 5C9422E4
-P 10000 4450
-F 0 "Q2" H 10206 4496 50  0000 L CNN
-F 1 "BSP75" H 10206 4405 50  0000 L CNN
-F 2 "Package_TO_SOT_SMD:SOT-223-3_TabPin2" H 10200 4375 50  0001 L CIN
-F 3 "" H 10200 4525 50  0001 L CNN
-	1    10000 4450
-	-1   0    0    1
-$EndComp
-Text HLabel 10500 4450 2    50   Input ~ 0
+P 9800 4450
+F 0 "Q2" H 10006 4496 50  0000 L CNN
+F 1 "BSP75" H 10006 4405 50  0000 L CNN
+F 2 "Package_TO_SOT_SMD:SOT-223-3_TabPin3" H 10000 4375 50  0001 L CIN
+F 3 "" H 10000 4525 50  0001 L CNN
+	1    9800 4450
+	1    0    0    -1
+$EndComp
+Text HLabel 9450 4450 1    50   Input ~ 0
 Sensor2_ON
 Wire Wire Line
@@
 L Device:R R4
 U 1 1 5C63383D
-P 9300 2150
-F 0 "R4" H 9370 2196 50  0000 L CNN
-F 1 "4.7k" H 9370 2105 50  0000 L CNN
-F 2 "Resistor_SMD:R_0805_2012Metric_Pad1.15x1.40mm_HandSolder" V 9230 2150 50  0001 C CNN
-F 3 "~" H 9300 2150 50  0001 C CNN
-	1    9300 2150
+P 9000 2150
+F 0 "R4" H 9070 2196 50  0000 L CNN
+F 1 "4.7k" H 9070 2105 50  0000 L CNN
+F 2 "Resistor_SMD:R_0805_2012Metric_Pad1.15x1.40mm_HandSolder" V 8930 2150 50  0001 C CNN
+F 3 "~" H 9000 2150 50  0001 C CNN
+	1    9000 2150
 	1    0    0    -1
 $EndComp
@@
 	9900 2550 9900 2600
 Wire Wire Line
-	10450 2350 10200 2350
-Wire Wire Line
-	9300 2000 9300 1650
-Wire Wire Line
-	9300 1650 9450 1650
-Wire Wire Line
-	9300 2300 9300 2600
-Wire Wire Line
-	9300 2600 9900 2600
+	9000 2000 9000 1650
+Wire Wire Line
+	9000 2300 9000 2600
 Connection ~ 9900 2600
 Wire Wire Line
@@
 	9200 3250 9900 3250
 Wire Wire Line
-	9050 3750 9300 3750
+	9050 3750 9100 3750
 Wire Wire Line
 	9900 4650 9900 4700
@@
 Connection ~ 9900 3250
 Wire Wire Line
-	10500 4450 10200 4450
-Wire Wire Line
-	9900 4700 9300 4700
-Wire Wire Line
-	9300 4700 9300 4250
+	9100 4700 9100 4250
 Connection ~ 9900 4700
 Wire Wire Line
 	9900 4700 9900 4750
 Wire Wire Line
-	9300 3950 9300 3750
-Connection ~ 9300 3750
-Wire Wire Line
-	9300 3750 9450 3750
-Connection ~ 9300 1650
-Wire Wire Line
-	8950 1650 9300 1650
+	9100 3950 9100 3750
 $Comp
 L Device:C C5
@@
 	6500 3000 6800 3000
 $Comp
-L Connector:Conn_01x01_Female J8
-U 1 1 5C897406
-P 3100 2450
-F 0 "J8" H 3127 2476 50  0000 L CNN
-F 1 "hole" H 3127 2385 50  0000 L CNN
-F 2 "MountingHole:MountingHole_3.2mm_M3" H 3100 2450 50  0001 C CNN
-F 3 "~" H 3100 2450 50  0001 C CNN
-	1    3100 2450
-	1    0    0    -1
-$EndComp
-$Comp
-L Connector:Conn_01x01_Female J9
-U 1 1 5C897463
-P 3100 2650
-F 0 "J9" H 3127 2676 50  0000 L CNN
-F 1 "hole" H 3127 2585 50  0000 L CNN
-F 2 "MountingHole:MountingHole_3.2mm_M3" H 3100 2650 50  0001 C CNN
-F 3 "~" H 3100 2650 50  0001 C CNN
-	1    3100 2650
-	1    0    0    -1
-$EndComp
-$Comp
-L Connector:Conn_01x01_Female J10
-U 1 1 5C8974BE
-P 3100 2850
-F 0 "J10" H 3127 2876 50  0000 L CNN
-F 1 "hole" H 3127 2785 50  0000 L CNN
-F 2 "MountingHole:MountingHole_3.2mm_M3" H 3100 2850 50  0001 C CNN
-F 3 "~" H 3100 2850 50  0001 C CNN
-	1    3100 2850
-	1    0    0    -1
-$EndComp
-$Comp
-L Connector:Conn_01x01_Female J11
-U 1 1 5C89751A
-P 3100 3050
-F 0 "J11" H 3127 3076 50  0000 L CNN
-F 1 "hole" H 3127 2985 50  0000 L CNN
-F 2 "MountingHole:MountingHole_3.2mm_M3" H 3100 3050 50  0001 C CNN
-F 3 "~" H 3100 3050 50  0001 C CNN
-	1    3100 3050
-	1    0    0    -1
-$EndComp
-NoConn ~ 2900 2450
-NoConn ~ 2900 2650
-NoConn ~ 2900 2850
-NoConn ~ 2900 3050
-$Comp
 L Hackuarium:LOGO G1
 U 1 1 5C89821B
@@
 	4000 1700 4450 1700
 $Comp
-L power:VCC #PWR?
+L power:VCC #PWR0105
 U 1 1 5CB91526
 P 1550 750
-F 0 "#PWR?" H 1550 600 50  0001 C CNN
+F 0 "#PWR0105" H 1550 600 50  0001 C CNN
 F 1 "VCC" H 1567 923 50  0000 C CNN
 F 2 "" H 1550 750 50  0001 C CNN
@@
 $EndComp
 $Comp
-L power:VCC #PWR?
+L power:VCC #PWR0106
 U 1 1 5CB998B1
 P 6500 850
-F 0 "#PWR?" H 6500 700 50  0001 C CNN
+F 0 "#PWR0106" H 6500 700 50  0001 C CNN
 F 1 "VCC" H 6517 1023 50  0000 C CNN
 F 2 "" H 6500 850 50  0001 C CNN
@@
 	1    0    0    -1
 $EndComp
+Connection ~ 9100 3750
+Wire Wire Line
+	9100 3750 9450 3750
+Wire Wire Line
+	9100 4700 9900 4700
+Wire Wire Line
+	9450 4450 9600 4450
+Wire Wire Line
+	8950 1650 9000 1650
+Connection ~ 9000 1650
+Wire Wire Line
+	9000 1650 9450 1650
+Wire Wire Line
+	9000 2600 9900 2600
+Wire Wire Line
+	9450 2350 9600 2350
 $EndSCHEMATC
