File: kicad/gas-sensor.kicad_pcb (KiCad board)
At the start: 2 copper layers, 100 x 100 mm, 37 parts, among them J1 Conn FT232RL, J2 RJ12, J3 hole, J4 hole, J5 hole, J6 hole, J7 5V_Power_source, Q1 BSP75, Q2 BSP75, U1 DS18B20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

Commit message: Update
Parts:
- C7: value 10u -> 10uF
- R1: value 1M -> 1MΩ
- R2: value 4,7 -> 4,7Ω
- R3, R5: value 10k -> 10kΩ
- R4: value 4.7k -> 4.7kΩ
- R6: value 4,7k -> 4,7kΩ
- U4: value MCP1703A-1202_SOT23 -> MCP1703A
- moved D2 3.95 mm to (123.9, 138.0)
- moved D1 3.89 mm to (123.9, 141.9)
- moved G1 2.32 mm to (140.1, 122.6)
- moved RV1 0.47 mm to (82.8, 145.9)
Routing:
- net /VCC-FTDI: track 76.3 -> 73.7 mm
- net Net-(C7-Pad1): track 16.3 -> 15.6 mm
- net /Sensor2_ON: track 16.9 -> 17.6 mm
- net /HUM: track 87.1 -> 87.8 mm
- net /PWM_MH-Z19: track 69.2 -> 69.8 mm
- net /LCD3_MISO: track 45.2 -> 45.8 mm
Other:
- board text added: "-1202_SOT23"
- board text added: "Gas sensor v1.2.0"
- board text removed: "Gas sensor v1.1.0"
