File: kicad/gas-sensor.kicad_pcb (KiCad board)
At the start: 2 copper layers, 100 x 100 mm, 37 parts, among them J1 Conn FT232RL, J2 RJ12, J3 hole, J4 hole, J5 hole, J6 hole, J7 5V_Power_source, Q1 BSP75, Q2 BSP75, U1 DS18B20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

Commit message: Update
Parts:
- moved GS3 0.18 mm to (90.4, 80.5)
Changed lines of the file:
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@@
-    )
-  )
-  (module footprints:MH-Z19 (layer F.Cu)
-    (at 90.25 80.37 270)
-    (fp_text reference GS3 (at 0 4 270) (layer F.Fab)
-      (effects (font (size 1 1) (thickness 0.15)))
-    )
-    (fp_text value MH-Z19 (at 0 -3 270) (layer F.SilkS)
-      (effects (font (size 1 1) (thickness 0.15)))
-    )
-    (fp_line (start -16.085 6.27) (end -13.25 6.27) (layer F.SilkS) (width 0.15))
-    (fp_line (start -16.085 -3.73) (end -13.25 -3.73) (layer F.SilkS) (width 0.15))
-    (fp_line (start 16.085 6.5) (end 13.25 6.5) (layer F.SilkS) (width 0.15))
-    (fp_line (start 16.085 -6.5) (end 13.25 -6.5) (layer F.SilkS) (width 0.15))
-    (fp_line (start 16.085 -6.5) (end 16.085 6.5) (layer F.SilkS) (width 0.15))
-    (fp_line (start -16.085 -3.73) (end -16.085 6.27) (layer F.SilkS) (width 0.15))
-    (fp_line (start -13.25 9.75) (end 13.25 9.75) (layer F.SilkS) (width 0.15))
-    (fp_line (start -13.25 -9.75) (end -13.25 9.75) (layer F.SilkS) (width 0.15))
-    (fp_line (start 13.25 -9.75) (end -13.25 -9.75) (layer F.SilkS) (width 0.15))
-    (fp_line (start 13.25 9.75) (end 13.25 -9.75) (layer F.SilkS) (width 0.15))
-    (pad 9 thru_hole circle (at -14.775 -2.54 270) (size 1.5 1.5) (drill 1) (layers *.Cu *.Mask)
-      (net 18 /PWM_MH-Z19))
-    (pad 8 thru_hole circle (at -14.775 0 270) (size 1.5 1.5) (drill 1) (layers *.Cu *.Mask))
-    (pad 7 thru_hole circle (at -14.775 2.54 270) (size 1.5 1.5) (drill 1) (layers *.Cu *.Mask)
-      (net 1 GND))
-    (pad 1 thru_hole circle (at 14.775 5.08 270) (size 1.5 1.5) (drill 1) (layers *.Cu *.Mask))
-    (pad 2 thru_hole circle (at 14.775 2.54 270) (size 1.5 1.5) (drill 1) (layers *.Cu *.Mask)
-      (net 16 /TX_MH-Z19))
-    (pad 3 thru_hole circle (at 14.775 0 270) (size 1.5 1.5) (drill 1) (layers *.Cu *.Mask)
-      (net 19 /RX_MH-Z19))
-    (pad 4 thru_hole circle (at 14.775 -2.54 270) (size 1.5 1.5) (drill 1) (layers *.Cu *.Mask))
-    (pad 5 thru_hole circle (at 14.775 -5.08 270) (size 1.5 1.5) (drill 1) (layers *.Cu *.Mask))
-    (pad 6 thru_hole circle (at -14.775 5.08 270) (size 1.5 1.5) (drill 1) (layers *.Cu *.Mask)
-      (net 7 +5V))
-    (model ${KIPRJMOD}/shapes3D/MH-Z19.wrl
-      (at (xyz 0 0 0))
-      (scale (xyz 400 400 400))
-      (rotate (xyz -90 0 0))
     )
   )
@@
     )
   )
+  (module footprints:MH-Z19 (layer F.Cu)
+    (at 90.41 80.45 270)
+    (fp_text reference GS3 (at 0 4 270) (layer F.SilkS)
+      (effects (font (size 1 1) (thickness 0.15)))
+    )
+    (fp_text value MH-Z19 (at 0 -3 270) (layer F.Fab)
+      (effects (font (size 1 1) (thickness 0.15)))
+    )
+    (fp_line (start 13.25 9.75) (end 13.25 -9.75) (layer F.SilkS) (width 0.15))
+    (fp_line (start 13.25 -9.75) (end -13.25 -9.75) (layer F.SilkS) (width 0.15))
+    (fp_line (start -13.25 -9.75) (end -13.25 9.75) (layer F.SilkS) (width 0.15))
+    (fp_line (start -13.25 9.75) (end 13.25 9.75) (layer F.SilkS) (width 0.15))
+    (fp_line (start -16.085 -3.73) (end -16.085 6.27) (layer F.SilkS) (width 0.15))
+    (fp_line (start 16.085 -6.5) (end 16.085 6.5) (layer F.SilkS) (width 0.15))
+    (fp_line (start 16.085 -6.5) (end 13.25 -6.5) (layer F.SilkS) (width 0.15))
+    (fp_line (start 16.085 6.5) (end 13.25 6.5) (layer F.SilkS) (width 0.15))
+    (fp_line (start -16.085 -3.73) (end -13.25 -3.73) (layer F.SilkS) (width 0.15))
+    (fp_line (start -16.085 6.27) (end -13.25 6.27) (layer F.SilkS) (width 0.15))
+    (pad 6 thru_hole circle (at -14.775 5.08 270) (size 1.5 1.5) (drill 1) (layers *.Cu *.Mask)
+      (net 7 +5V))
+    (pad 5 thru_hole circle (at 14.775 -5.08 270) (size 1.5 1.5) (drill 1) (layers *.Cu *.Mask))
+    (pad 4 thru_hole circle (at 14.775 -2.54 270) (size 1.5 1.5) (drill 1) (layers *.Cu *.Mask))
+    (pad 3 thru_hole circle (at 14.775 0 270) (size 1.5 1.5) (drill 1) (layers *.Cu *.Mask)
+      (net 19 /RX_MH-Z19))
+    (pad 2 thru_hole circle (at 14.775 2.54 270) (size 1.5 1.5) (drill 1) (layers *.Cu *.Mask)
+      (net 16 /TX_MH-Z19))
+    (pad 1 thru_hole circle (at 14.775 5.08 270) (size 1.5 1.5) (drill 1) (layers *.Cu *.Mask))
+    (pad 7 thru_hole circle (at -14.775 2.54 270) (size 1.5 1.5) (drill 1) (layers *.Cu *.Mask)
+      (net 1 GND))
+    (pad 8 thru_hole circle (at -14.775 0 270) (size 1.5 1.5) (drill 1) (layers *.Cu *.Mask))
+    (pad 9 thru_hole circle (at -14.775 -2.54 270) (size 1.5 1.5) (drill 1) (layers *.Cu *.Mask)
+      (net 18 /PWM_MH-Z19))
+    (model ${KIPRJMOD}/shapes3D/MH-Z19.STEP
+      (at (xyz 0 0 0))
+      (scale (xyz 1 1 1))
+      (rotate (xyz -90 0 0))
+    )
+  )
   (gr_text -1202_SOT23 (at 132.11 134.78) (layer F.SilkS)
     (effects (font (size 0.63 0.63) (thickness 0.13)))
@@
   (gr_line (start 145 102.25) (end 55 102.25) (layer F.SilkS) (width 0.2))
   (gr_line (start 55 58.25) (end 145 58.25) (layer F.SilkS) (width 0.2))
+  (segment (start 93.917934 126.012755) (end 93.917934 125.287934) (width 0.5) (layer F.Cu) (net 0))
   (segment (start 93.552936 130.662755) (end 92.467934 130.662755) (width 0.5) (layer F.Cu) (net 1) (status 20))
   (segment (start 93.717935 130.497756) (end 93.552936 130.662755) (width 0.5) (layer F.Cu) (net 1))
@@
   (segment (start 103.127245 129.062755) (end 103.45 128.74) (width 0.5) (layer F.Cu) (net 12))
   (segment (start 100.967934 129.062755) (end 103.127245 129.062755) (width 0.5) (layer F.Cu) (net 12))
-  (segment (start 93.917934 126.012755) (end 93.917934 125.287934) (width 0.5) (layer F.Cu) (net 0))
   (via (at 94.15 127.8) (size 0.8) (drill 0.4) (layers F.Cu B.Cu) (net 13))
   (segment (start 93.687245 128.262755) (end 94.15 127.8) (width 0.5) (layer F.Cu) (net 13))
@@
   (segment (start 91.645183 121.640004) (end 57.359996 121.640004) (width 0.5) (layer F.Cu) (net 15))
   (segment (start 94.717934 124.712755) (end 91.645183 121.640004) (width 0.5) (layer F.Cu) (net 15))
-  (segment (start 98.717934 126.012755) (end 98.717934 123.575417) (width 0.5) (layer F.Cu) (net 16) (status 10))
+  (segment (start 100.94 108.295) (end 87.87 95.225) (width 0.5) (layer F.Cu) (net 16))
+  (segment (start 100.94 121.353351) (end 100.94 108.295) (width 0.5) (layer F.Cu) (net 16))
   (segment (start 98.717934 123.575417) (end 100.94 121.353351) (width 0.5) (layer F.Cu) (net 16))
-  (segment (start 100.94 108.375) (end 100.94 121.353351) (width 0.5) (layer F.Cu) (net 16))
-  (segment (start 87.71 95.145) (end 100.94 108.375) (width 0.5) (layer F.Cu) (net 16) (status 10))
+  (segment (start 98.717934 126.012755) (end 98.717934 123.575417) (width 0.5) (layer F.Cu) (net 16))
   (segment (start 108.535 89.58) (end 109.56 89.58) (width 0.5) (layer F.Cu) (net 17))
   (segment (start 104.8 93.315) (end 108.535 89.58) (width 0.5) (layer F.Cu) (net 17))
@@
   (segment (start 80.21 145.995) (end 80.21 140.200689) (width 1) (layer F.Cu) (net 17))
   (via (at 90.92 114.58) (size 0.8) (drill 0.4) (layers F.Cu B.Cu) (net 18))
-  (segment (start 83.969999 107.859999) (end 83.969999 74.415001) (width 0.5) (layer F.Cu) (net 18))
-  (segment (start 84.199999 107.859999) (end 83.969999 107.859999) (width 0.5) (layer F.Cu) (net 18))
-  (segment (start 83.969999 74.415001) (end 92.79 65.595) (width 0.5) (layer F.Cu) (net 18) (status 20))
-  (segment (start 90.92 114.58) (end 84.199999 107.859999) (width 0.5) (layer F.Cu) (net 18))
   (segment (start 90.92 114.58) (end 90.92 122.490014) (width 0.5) (layer B.Cu) (net 18))
   (via (at 90.92 122.490014) (size 0.8) (drill 0.4) (layers F.Cu B.Cu) (net 18))
@@
   (segment (start 91.482755 127.462755) (end 90.92 126.9) (width 0.5) (layer F.Cu) (net 18))
   (segment (start 92.467934 127.462755) (end 91.482755 127.462755) (width 0.5) (layer F.Cu) (net 18))
-  (segment (start 99.517934 123.765382) (end 99.517934 126.012755) (width 0.5) (layer F.Cu) (net 19) (status 20))
-  (segment (start 101.640011 121.643305) (end 99.517934 123.765382) (width 0.5) (layer F.Cu) (net 19))
-  (segment (start 101.640011 106.570011) (end 101.640011 121.643305) (width 0.5) (layer F.Cu) (net 19))
-  (segment (start 90.25 95.18) (end 101.640011 106.570011) (width 0.5) (layer F.Cu) (net 19) (status 10))
+  (segment (start 83.969999 74.655001) (end 92.95 65.675) (width 0.5) (layer F.Cu) (net 18))
+  (segment (start 83.969999 107.859999) (end 83.969999 74.655001) (width 0.5) (layer F.Cu) (net 18))
+  (segment (start 84.199999 107.859999) (end 83.969999 107.859999) (width 0.5) (layer F.Cu) (net 18))
+  (segment (start 90.92 114.58) (end 84.199999 107.859999) (width 0.5) (layer F.Cu) (net 18))
   (segment (start 90.25 95.145) (end 90.25 95.18) (width 0.5) (layer F.Cu) (net 19) (status 30))
+  (segment (start 101.640011 106.455011) (end 90.41 95.225) (width 0.5) (layer F.Cu) (net 19))
+  (segment (start 101.640011 121.643305) (end 101.640011 106.455011) (width 0.5) (layer F.Cu) (net 19))
+  (segment (start 99.517934 123.765382) (end 101.640011 121.643305) (width 0.5) (layer F.Cu) (net 19))
+  (segment (start 99.517934 126.012755) (end 99.517934 123.765382) (width 0.5) (layer F.Cu) (net 19))
   (via (at 81.5 137.98) (size 0.8) (drill 0.4) (layers F.Cu B.Cu) (net 20))
   (via (at 78.41 137.98) (size 0.8) (drill 0.4) (layers F.Cu B.Cu) (net 20))
